File: macropad-practice.kicad_sch (KiCad schematic)
At the start: 14 parts, among them SW1 RotaryEncoder_Switch, SW2 SW_Push, SW3 SW_Push, SW4 SW_Push, SW5 SW_MEC_5E, SW6 SW_Push, SW7 SW_Push, U1 ProMicro

Commit message: routing done
Parts:
- SW5: footprint Button_Switch_SMD:SW_SPST_SKQG_WithStem -> random-keyboard-parts:PushButton_6x6mm_TH
Connections:
- net COL0: now also U1.16 (B1)
- net COL1: now also U1.15 (B3)
- net ENCA: now also U1.13 (B6)
- net ENCB: now also U1.14 (B2)
- net ROW0: now also U1.5 (SDA)
- net ROW1: now also U1.6 (SCL)
- net ROW2: now also U1.7 (D4)
- no-connect marks 0 -> 5
Changed lines of the file:
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@@
   (junction (at 147.32 81.28) (diameter 0) (color 0 0 0 0)
   )
+  (no_connect (at 218.44 49.53))
+  (no_connect (at 254 46.99))
+  (no_connect (at 276.86 63.5))
+  (no_connect (at 266.7 63.5))
+  (no_connect (at 218.44 46.99))
   (wire (pts (xy 171.45 13.97) (xy 179.07 13.97))
     (stroke (width 0) (type default) (color 0 0 0 0))
@@
     (stroke (width 0) (type default) (color 0 0 0 0))
   )
+  (global_label "ENCA" (shape input) (at 254 74.93 0) (fields_autoplaced)
+    (effects (font (size 1.27 1.27)) (justify left))
+    (property "Intersheet References" "${INTERSHEET_REFS}" (id 0) (at 261.2512 74.8506 0)
+      (effects (font (size 1.27 1.27)) (justify left) hide)
+    )
+  )
   (global_label "ENCA" (shape input) (at 173.99 26.67 90) (fields_autoplaced)
     (effects (font (size 1.27 1.27)) (justify left))
     (property "Intersheet References" "${INTERSHEET_REFS}" (id 0) (at 173.9106 19.4188 90)
+      (effects (font (size 1.27 1.27)) (justify left) hide)
+    )
+  )
+  (global_label "ROW0" (shape input) (at 218.44 57.15 180) (fields_autoplaced)
+    (effects (font (size 1.27 1.27)) (justify right))
+    (property "Intersheet References" "${INTERSHEET_REFS}" (id 0) (at 210.7655 57.0706 0)
+      (effects (font (size 1.27 1.27)) (justify right) hide)
+    )
+  )
+  (global_label "ENCB" (shape input) (at 254 72.39 0) (fields_autoplaced)
+    (effects (font (size 1.27 1.27)) (justify left))
+    (property "Intersheet References" "${INTERSHEET_REFS}" (id 0) (at 261.4326 72.3106 0)
       (effects (font (size 1.27 1.27)) (justify left) hide)
     )
@@
     )
   )
+  (global_label "ROW2" (shape input) (at 218.44 62.23 180) (fields_autoplaced)
+    (effects (font (size 1.27 1.27)) (justify right))
+    (property "Intersheet References" "${INTERSHEET_REFS}" (id 0) (at 210.7655 62.1506 0)
+      (effects (font (size 1.27 1.27)) (justify right) hide)
+    )
+  )
+  (global_label "ROW1" (shape input) (at 218.44 59.69 180) (fields_autoplaced)
+    (effects (font (size 1.27 1.27)) (justify right))
+    (property "Intersheet References" "${INTERSHEET_REFS}" (id 0) (at 210.7655 59.6106 0)
+      (effects (font (size 1.27 1.27)) (justify right) hide)
+    )
+  )
+  (global_label "COL0" (shape input) (at 254 67.31 0) (fields_autoplaced)
+    (effects (font (size 1.27 1.27)) (justify left))
+    (property "Intersheet References" "${INTERSHEET_REFS}" (id 0) (at 261.2512 67.3894 0)
+      (effects (font (size 1.27 1.27)) (justify left) hide)
+    )
+  )
   (global_label "ROW2" (shape input) (at 138.43 81.28 180) (fields_autoplaced)
     (effects (font (size 1.27 1.27)) (justify right))
@@
     )
   )
+  (global_label "COL1" (shape input) (at 254 69.85 0) (fields_autoplaced)
+    (effects (font (size 1.27 1.27)) (justify left))
+    (property "Intersheet References" "${INTERSHEET_REFS}" (id 0) (at 261.2512 69.9294 0)
+      (effects (font (size 1.27 1.27)) (justify left) hide)
+    )
+  )
   (symbol (lib_id "Switch:SW_MEC_5E") (at 271.78 60.96 180) (unit 1)
     (in_bom yes) (on_board yes) (fields_autoplaced)
     (property "Reference" "SW5" (id 0) (at 271.78 55.88 0))
     (property "Value" "SW_MEC_5E" (id 1) (at 271.78 58.42 0))
-    (property "Footprint" "Button_Switch_SMD:SW_SPST_SKQG_WithStem" (id 2) (at 271.78 68.58 0)
+    (property "Footprint" "random-keyboard-parts:PushButton_6x6mm_TH" (id 2) (at 271.78 68.58 0)
       (effects (font (size 1.27 1.27)) hide)
     )
@@
     )
     (path "/1e5778a0-aa39-4ebf-8ee2-3c036592f77d"
-      (reference "SW5") (unit 1) (value "SW_MEC_5E") (footprint "Button_Switch_SMD:SW_SPST_SKQG_WithStem")
+      (reference "SW5") (unit 1) (value "SW_MEC_5E") (footprint "random-keyboard-parts:PushButton_6x6mm_TH")
     )
     (path "/6c1c409b-9c5b-40f9-b41e-75318bbd679f"
