File: macropad-practice.kicad_pcb (KiCad board)
At the start: 2 copper layers, 106.6 x 98.5 mm, 14 parts, among them SW1 RotaryEncoder_Switch, SW2 SW_Push, SW3 SW_Push, SW4 SW_Push, SW5 SW_MEC_5E, SW6 SW_Push, SW7 SW_Push, U1 ProMicro

Commit message: added some details
Routing:
- net COL0: track 151.2 -> 149.8 mm
- net ROW0: track 9.52 -> 8.62 mm
Other:
- board text added: "Pentakill v0.1"
- board text added: "by Teckt"
Changed lines of the file:
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@@
   (gr_arc (start 91.28125 115.093749) (mid 88.378623 112.576313) (end 88.106251 108.74375) (layer "Edge.Cuts") (width 0.1))
   (gr_arc (start 101.219001 46.355) (mid 101.689859 45.196354) (end 102.697393 44.45538) (layer "Edge.Cuts") (width 0.1))
+  (gr_text "Pentakill v0.1" (at 140.589 100.33) (layer "F.SilkS")
+    (effects (font (size 2 2) (thickness 0.3)))
+  )
+  (gr_text "by Teckt" (at 147.955 102.743) (layer "F.SilkS")
+    (effects (font (size 1 1) (thickness 0.15)))
+  )
   (segment (start 153.925 55.5625) (end 153.925 58.293) (width 0.254) (layer "F.Cu") (net 1))
-  (segment (start 148.74875 58.7375) (end 148.11375 58.1025) (width 0.254) (layer "F.Cu") (net 1))
   (segment (start 153.925 58.293) (end 148.30425 58.293) (width 0.254) (layer "F.Cu") (net 1))
   (segment (start 148.30425 58.293) (end 148.11375 58.1025) (width 0.254) (layer "F.Cu") (net 1))
@@
   (segment (start 125.476 69.596) (end 126.8095 68.2625) (width 0.254) (layer "F.Cu") (net 14))
   (segment (start 105.6875 93.925) (end 106.481 93.925) (width 0.254) (layer "F.Cu") (net 14))
-  (segment (start 172.3625 51.85625) (end 171.410989 50.904739) (width 0.254) (layer "B.Cu") (net 14))
   (segment (start 113.625 51.85625) (end 113.625 51.31625) (width 0.254) (layer "B.Cu") (net 14))
   (segment (start 113.625 51.31625) (end 113.665 51.27625) (width 0.254) (layer "B.Cu") (net 14))
@@
   (zone (net 12) (net_name "GND") (layer "B.Cu") (hatch edge 0.508)
     (connect_pads (clearance 0.508))
-    (min_thickness 0.254)
-    (fill (thermal_gap 0.508) (thermal_bridge_width 0.508))
+    (min_thickness 0.254) (filled_areas_thickness no)
+    (fill yes (thermal_gap 0.508) (thermal_bridge_width 0.508))
     (polygon
       (pts
